File: mp3/mp3.kicad_sch (KiCad schematic)
At the start: 46 parts, among them J1 Micro_SD_Card, J2 USB_C_Receptacle_PowerOnly_6P, J3 AudioPlug3, J4 Conn_01x04, SW1 POWER, SW2 VOL -, SW3 VOL +, SW4 NEXT, SW5 PREV, SW6 PLAY, U1 ESP32-S3-WROOM-1, U2 PCM5102A, U3 TPA6132A2RTE, U4 BQ24074RGT

Commit message: changed pcb
Connections:
- net GND: now also SW2.2, SW3.2, SW4.2, SW5.2, SW6.2
- net at U1.33 (IO40): now also SW4.1; no longer SW6.2
- new net: SW2.1, U1.31 (IO38)
- new net: SW3.1, U1.32 (IO39)
- new net: SW5.1, U1.34 (IO41)
- new net: SW6.1, U1.35 (IO42)
Other:
- moved on the sheet: SW2, SW3, SW4, SW5, SW6
