File: mp3/mp3.kicad_pcb (KiCad board)
At the start: 2 copper layers, 53 x 36 mm, 47 parts, among them J1 Micro_SD_Card, J2 USB_C_Receptacle_PowerOnly_6P, J3 AudioPlug3, J4 Conn_01x04, SW1 POWER, SW2 VOL -, SW3 VOL +, SW4 NEXT, SW5 PREV, SW6 PLAY, U1 ESP32-S3-WROOM-1, U2 PCM5102A, U3 TPA6132A2RTE, U4 BQ24074RGT

Commit message: more pcb changes
Parts:
- moved SW3 3.54 mm to (168.5, 92.0), turned to 180 degrees
- moved SW2 2.92 mm to (166.5, 92.0), turned to 0 degrees
- moved SW5 2.55 mm to (168.5, 93.0), turned to 180 degrees
- moved SW6 2.12 mm to (166.5, 94.0), turned to 0 degrees
- moved SW4 1.58 mm to (166.5, 93.0), turned to 0 degrees
Connections:
- SW2 pad 1: Net-(U1-IO41) -> Net-(U1-IO38)
- SW2 pad 2: Net-(U1-IO38) -> GND
- SW3 pad 1: Net-(U1-IO42) -> Net-(U1-IO39)
- SW3 pad 2: Net-(U1-IO38) -> GND
- SW4 pad 1: Net-(U1-IO41) -> Net-(U1-IO40)
- SW4 pad 2: Net-(U1-IO39) -> GND
- SW5 pad 1: Net-(U1-IO42) -> Net-(U1-IO41)
- SW5 pad 2: Net-(U1-IO39) -> GND
- SW6 pad 1: Net-(U1-IO41) -> Net-(U1-IO42)
- SW6 pad 2: Net-(U1-IO40) -> GND
Routing:
- net Net-(U1-IO40): track 19.4 -> 24.6 mm
- net GND: track 185.9 -> 190.9 mm
- net Net-(U1-IO42): track 26.1 -> 28.5 mm
- net Net-(U1-IO41): track 21.5 -> 23.8 mm
- net Net-(U1-IO39): track 21.9 -> 20.1 mm, vias 3 -> 1
- net Net-(U1-IO38): track 21.2 -> 19.9 mm
- net Net-(J1-DAT3/CD): track 31.9 -> 32.6 mm
